File: pcb/wifi_ledstrip/schematic.brd (EAGLE design)
At the start: 80 x 49.5 mm, 65 parts, among them IC1 STM32F10XCXT6, Q1 8MHz

Commit message: pcb updated with leds
Parts:
- HEARTBEAT: value GREEN -> RED
- L_12V: value GREEN -> WHITE
- L_3V3: value GREEN -> BLUE
- L_5V: value GREEN -> ORANGE
- L_TX: value GREEN -> YELLOW
- R2, R3, R4, R5, R7: value (none) -> 62R
Changed lines of the file:
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@@
 <drawing>
 <settings>
-<setting alwaysvectorfont="yes"/>
+<setting alwaysvectorfont="no"/>
 <setting verticaltext="up"/>
 </settings>
@@
 <attribute name="VALUE" x="11.57" y="5.52" size="0.6096" layer="27" font="vector" ratio="20"/>
 </element>
-<element name="L_12V" library="SparkFun-LED" library_urn="urn:adsk.eagle:library:529" package="LED-1206" package3d_urn="urn:adsk.eagle:package:39352/1" value="GREEN" x="8.2" y="8.25" smashed="yes" rot="R270">
+<element name="L_12V" library="SparkFun-LED" library_urn="urn:adsk.eagle:library:529" package="LED-1206" package3d_urn="urn:adsk.eagle:package:39352/1" value="WHITE" x="8.2" y="8.25" smashed="yes" rot="R270">
 <attribute name="NAME" x="9.1525" y="8.25" size="0.6096" layer="25" font="vector" ratio="20" rot="R270" align="bottom-center"/>
 <attribute name="PROD_ID" value="DIO-00862" x="8.2" y="8.25" size="1.778" layer="27" rot="R270" display="off"/>
 <attribute name="VALUE" x="7.2475" y="8.25" size="0.6096" layer="27" font="vector" ratio="20" rot="R270" align="top-center"/>
 </element>
-<element name="L_5V" library="SparkFun-LED" library_urn="urn:adsk.eagle:library:529" package="LED-1206" package3d_urn="urn:adsk.eagle:package:39352/1" value="GREEN" x="5.7" y="8.27" smashed="yes" rot="R270">
+<element name="L_5V" library="SparkFun-LED" library_urn="urn:adsk.eagle:library:529" package="LED-1206" package3d_urn="urn:adsk.eagle:package:39352/1" value="ORANGE" x="5.7" y="8.27" smashed="yes" rot="R270">
 <attribute name="NAME" x="6.6525" y="8.27" size="0.6096" layer="25" font="vector" ratio="20" rot="R270" align="bottom-center"/>
 <attribute name="PROD_ID" value="DIO-00862" x="5.7" y="8.27" size="1.778" layer="27" rot="R270" display="off"/>
 <attribute name="VALUE" x="4.7475" y="8.27" size="0.6096" layer="27" font="vector" ratio="20" rot="R270" align="top-center"/>
 </element>
-<element name="L_3V3" library="SparkFun-LED" library_urn="urn:adsk.eagle:library:529" package="LED-1206" package3d_urn="urn:adsk.eagle:package:39352/1" value="GREEN" x="3.14" y="8.27" smashed="yes" rot="R270">
+<element name="L_3V3" library="SparkFun-LED" library_urn="urn:adsk.eagle:library:529" package="LED-1206" package3d_urn="urn:adsk.eagle:package:39352/1" value="BLUE" x="3.14" y="8.27" smashed="yes" rot="R270">
 <attribute name="NAME" x="4.0925" y="8.27" size="0.6096" layer="25" font="vector" ratio="20" rot="R270" align="bottom-center"/>
 <attribute name="PROD_ID" value="DIO-00862" x="3.14" y="8.27" size="1.778" layer="27" rot="R270" display="off"/>
@@
 <attribute name="VALUE" x="43.35" y="25.7775" size="0.6096" layer="27" font="vector" ratio="20" align="top-center"/>
 </element>
-<element name="L_TX" library="SparkFun-LED" library_urn="urn:adsk.eagle:library:529" package="LED-1206" package3d_urn="urn:adsk.eagle:package:39352/1" value="GREEN" x="43.35" y="29.4" smashed="yes">
+<element name="L_TX" library="SparkFun-LED" library_urn="urn:adsk.eagle:library:529" package="LED-1206" package3d_urn="urn:adsk.eagle:package:39352/1" value="YELLOW" x="43.35" y="29.4" smashed="yes">
 <attribute name="NAME" x="43.35" y="30.3525" size="0.6096" layer="25" font="vector" ratio="20" align="bottom-center"/>
 <attribute name="PROD_ID" value="DIO-00862" x="43.35" y="29.4" size="1.778" layer="27" display="off"/>
 <attribute name="VALUE" x="43.35" y="28.4475" size="0.6096" layer="27" font="vector" ratio="20" align="top-center"/>
 </element>
-<element name="HEARTBEAT" library="SparkFun-LED" library_urn="urn:adsk.eagle:library:529" package="LED-1206" package3d_urn="urn:adsk.eagle:package:39352/1" value="GREEN" x="17.65" y="47.18" smashed="yes" rot="R180">
+<element name="HEARTBEAT" library="SparkFun-LED" library_urn="urn:adsk.eagle:library:529" package="LED-1206" package3d_urn="urn:adsk.eagle:package:39352/1" value="RED" x="17.65" y="47.18" smashed="yes" rot="R180">
 <attribute name="NAME" x="17.65" y="46.2275" size="0.6096" layer="25" font="vector" ratio="20" rot="R180" align="bottom-center"/>
 <attribute name="PROD_ID" value="DIO-00862" x="17.65" y="47.18" size="1.778" layer="27" rot="R180" display="off"/>
@@
 <attribute name="VALUE" x="8.31" y="9.23" size="1.27" layer="27"/>
 </element>
-<element name="R2" library="rcl" library_urn="urn:adsk.eagle:library:334" package="R1206" package3d_urn="urn:adsk.eagle:package:23540/2" value="" x="5.84" y="13.37" smashed="yes" rot="R90">
+<element name="R2" library="rcl" library_urn="urn:adsk.eagle:library:334" package="R1206" package3d_urn="urn:adsk.eagle:package:23540/2" value="62R" x="5.84" y="13.37" smashed="yes" rot="R90">
 <attribute name="NAME" x="6.44" y="15.88" size="1.27" layer="25" rot="R90"/>
 <attribute name="SPICEPREFIX" value="R" x="5.84" y="13.37" size="1.778" layer="27" rot="R90" display="off"/>
 <attribute name="VALUE" x="8.38" y="12.1" size="1.27" layer="27" rot="R90"/>
 </element>
-<element name="R3" library="rcl" library_urn="urn:adsk.eagle:library:334" package="R1206" package3d_urn="urn:adsk.eagle:package:23540/2" value="" x="3.17" y="13.37" smashed="yes" rot="R90">
+<element name="R3" library="rcl" library_urn="urn:adsk.eagle:library:334" package="R1206" package3d_urn="urn:adsk.eagle:package:23540/2" value="62R" x="3.17" y="13.37" smashed="yes" rot="R90">
 <attribute name="NAME" x="3.8" y="15.86" size="1.27" layer="25" rot="R90"/>
 <attribute name="SPICEPREFIX" value="R" x="3.17" y="13.37" size="1.778" layer="27" rot="R90" display="off"/>
 <attribute name="VALUE" x="5.71" y="12.1" size="1.27" layer="27" rot="R90"/>
 </element>
-<element name="R4" library="rcl" library_urn="urn:adsk.eagle:library:334" package="R1206" package3d_urn="urn:adsk.eagle:package:23540/2" value="" x="38.53" y="31.58" smashed="yes" rot="MR90">
+<element name="R4" library="rcl" library_urn="urn:adsk.eagle:library:334" package="R1206" package3d_urn="urn:adsk.eagle:package:23540/2" value="62R" x="38.53" y="31.58" smashed="yes" rot="MR90">
 <attribute name="NAME" x="39.8" y="29.9036" size="1.27" layer="26" rot="MR90"/>
 <attribute name="SPICEPREFIX" value="R" x="38.53" y="31.58" size="1.778" layer="28" rot="MR90" display="off"/>
 <attribute name="VALUE" x="35.99" y="30.31" size="1.27" layer="28" rot="MR90"/>
 </element>
-<element name="R5" library="rcl" library_urn="urn:adsk.eagle:library:334" package="R1206" package3d_urn="urn:adsk.eagle:package:23540/2" value="" x="34.7" y="31.58" smashed="yes" rot="MR90">
+<element name="R5" library="rcl" library_urn="urn:adsk.eagle:library:334" package="R1206" package3d_urn="urn:adsk.eagle:package:23540/2" value="62R" x="34.7" y="31.58" smashed="yes" rot="MR90">
 <attribute name="NAME" x="35.97" y="30.9196" size="1.27" layer="26" rot="MR90"/>
 <attribute name="SPICEPREFIX" value="R" x="34.7" y="31.58" size="1.778" layer="28" rot="MR90" display="off"/>
@@
 <attribute name="VALUE" x="66.8596" y="36.19" size="1.27" layer="27" rot="R270"/>
 </element>
-<element name="R7" library="rcl" library_urn="urn:adsk.eagle:library:334" package="R1206" package3d_urn="urn:adsk.eagle:package:23540/2" value="" x="23.42" y="47.29" smashed="yes" rot="R180">
+<element name="R7" library="rcl" library_urn="urn:adsk.eagle:library:334" package="R1206" package3d_urn="urn:adsk.eagle:package:23540/2" value="62R" x="23.42" y="47.29" smashed="yes" rot="R180">
 <attribute name="NAME" x="24.69" y="46.02" size="1.27" layer="25" rot="R180"/>
 <attribute name="SPICEPREFIX" value="R" x="23.42" y="47.29" size="1.778" layer="27" rot="R180" display="off"/>
